File: Hardware/PCB_kicad/laberinto.kicad_pcb (KiCad board)
At the start: 2 copper layers, 87.5 x 70 mm, 34 parts, among them IC1 L293D, P1 Digital, P10 distance, P11 M1, P12 M2, P3 ADC, P4 Analog, P6 batt, P7 buzzer, P8 I2C_IMU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

Commit message: Fixed track
Routing:
- net Net-(D1-Pad2): track 0.00 -> 9.63 mm
- net GND: track 248.5 -> 257.4 mm
